File: 74HC165.sch (KiCad schematic (older format))
At the start: 6 parts, among them J2 Conn_01x05, J3 Conn_01x05, U1 74HC165

Commit message: Put ground on pin 1 of all the connectors Fixes #1
Connections:
- net A: now also J2.2 (Pin_2); no longer J2.1 (Pin_1)
- net B: now also J2.3 (Pin_3); no longer J2.2 (Pin_2)
- net C: now also J2.4 (Pin_4); no longer J2.3 (Pin_3)
- net D: now also J2.5 (Pin_5); no longer J2.4 (Pin_4)
- net E: now also J3.2 (Pin_2); no longer J3.1 (Pin_1)
- net F: now also J3.3 (Pin_3); no longer J3.2 (Pin_2)
- net G: now also J3.4 (Pin_4); no longer J3.3 (Pin_3)
- net GND: now also J2.1 (Pin_1), J3.1 (Pin_1); no longer J2.5 (Pin_5), J3.5 (Pin_5)
- net H: now also J3.5 (Pin_5); no longer J3.4 (Pin_4)
Changed lines of the file:
@@
 $Descr A4 11693 8268
 encoding utf-8
-Sheet 2 5
+Sheet 4 5
 Title ""
 Date "%%date%%"
@@
 AR Path="/61DDC3C8/61DD4B9D" Ref="U3"  Part="1"
 AR Path="/61DDC5F2/61DD4B9D" Ref="U4"  Part="1"
-F 0 "U1" H 3350 3231 50  0000 C CNN
+F 0 "U3" H 3350 3231 50  0000 C CNN
 F 1 "74HC165" H 3350 3140 50  0000 C CNN
 F 2 "Package_SO:SOIC-16_3.9x9.9mm_P1.27mm" H 3350 2150 50  0001 C CNN
@@
 AR Path="/61DDC3C8/61DD4BA3" Ref="C3"  Part="1"
 AR Path="/61DDC5F2/61DD4BA3" Ref="C4"  Part="1"
-F 0 "C1" H 4292 1396 50  0000 L CNN
+F 0 "C3" H 4292 1396 50  0000 L CNN
 F 1 "100nF" H 4292 1305 50  0000 L CNN
 F 2 "Capacitor_SMD:C_0805_2012Metric" H 4200 1350 50  0001 C CNN
@@
 AR Path="/61DDC3C8/61DD4BEE" Ref="#PWR017"  Part="1"
 AR Path="/61DDC5F2/61DD4BEE" Ref="#PWR022"  Part="1"
-F 0 "#PWR07" H 3500 2900 50  0001 C CNN
+F 0 "#PWR017" H 3500 2900 50  0001 C CNN
 F 1 "GND" H 3505 2977 50  0000 C CNN
 F 2 "" H 3500 3150 50  0001 C CNN
@@
 AR Path="/61DDC3C8/61DD4BF6" Ref="#PWR013"  Part="1"
 AR Path="/61DDC5F2/61DD4BF6" Ref="#PWR018"  Part="1"
-F 0 "#PWR03" H 4200 1100 50  0001 C CNN
+F 0 "#PWR013" H 4200 1100 50  0001 C CNN
 F 1 "+5V" H 4215 1423 50  0000 C CNN
 F 2 "" H 4200 1250 50  0001 C CNN
@@
 AR Path="/61DDC3C8/61DD4BFD" Ref="#PWR014"  Part="1"
 AR Path="/61DDC5F2/61DD4BFD" Ref="#PWR019"  Part="1"
-F 0 "#PWR04" H 4200 1200 50  0001 C CNN
+F 0 "#PWR014" H 4200 1200 50  0001 C CNN
 F 1 "GND" H 4205 1277 50  0000 C CNN
 F 2 "" H 4200 1450 50  0001 C CNN
@@
 AR Path="/61DDC3C8/61DBAD50" Ref="RN6"  Part="1"
 AR Path="/61DDC5F2/61DBAD50" Ref="RN8"  Part="1"
-F 0 "RN2" H 2400 850 50  0000 C CNN
+F 0 "RN6" H 2400 850 50  0000 C CNN
 F 1 "R_Pack04" H 2400 950 50  0000 C CNN
 F 2 "Resistor_SMD:R_Array_Convex_4x0603" V 2725 1250 50  0001 C CNN
@@
 AR Path="/61DDC3C8/61DCA935" Ref="J7"  Part="1"
 AR Path="/61DDC5F2/61DCA935" Ref="J9"  Part="1"
-F 0 "J3" H 1500 2500 50  0000 R CNN
+F 0 "J7" H 1500 2500 50  0000 R CNN
 F 1 "Conn_01x05" H 1900 2400 50  0000 R CNN
 F 2 "Connector_JST:JST_XH_B5B-XH-A_1x05_P2.50mm_Vertical" H 1350 2400 50  0001 C CNN
@@
 	1    1350 2400
 	-1   0    0    -1
-$EndComp
-$Comp
-L power:GND #PWR06
-U 1 1 61DCA93B
-P 1550 2600
-AR Path="/61DCCBDC/61DCA93B" Ref="#PWR06"  Part="1"
-AR Path="/61DDC172/61DCA93B" Ref="#PWR011"  Part="1"
-AR Path="/61DDC3C8/61DCA93B" Ref="#PWR016"  Part="1"
-AR Path="/61DDC5F2/61DCA93B" Ref="#PWR021"  Part="1"
-F 0 "#PWR06" H 1550 2350 50  0001 C CNN
-F 1 "GND" H 1555 2427 50  0000 C CNN
-F 2 "" H 1550 2600 50  0001 C CNN
-F 3 "" H 1550 2600 50  0001 C CNN
-	1    1550 2600
-	1    0    0    -1
 $EndComp
 $Comp
@@
 AR Path="/61DDC3C8/61DCC07D" Ref="J6"  Part="1"
 AR Path="/61DDC5F2/61DCC07D" Ref="J8"  Part="1"
-F 0 "J2" H 1500 1800 50  0000 R CNN
+F 0 "J6" H 1500 1800 50  0000 R CNN
 F 1 "Conn_01x05" H 1900 1700 50  0000 R CNN
 F 2 "Connector_JST:JST_XH_B5B-XH-A_1x05_P2.50mm_Vertical" H 1350 1700 50  0001 C CNN
@@
 L power:GND #PWR05
 U 1 1 61DCC083
-P 1550 1900
+P 750 2650
 AR Path="/61DCCBDC/61DCC083" Ref="#PWR05"  Part="1"
 AR Path="/61DDC172/61DCC083" Ref="#PWR010"  Part="1"
 AR Path="/61DDC3C8/61DCC083" Ref="#PWR015"  Part="1"
 AR Path="/61DDC5F2/61DCC083" Ref="#PWR020"  Part="1"
-F 0 "#PWR05" H 1550 1650 50  0001 C CNN
-F 1 "GND" H 1555 1727 50  0000 C CNN
-F 2 "" H 1550 1900 50  0001 C CNN
-F 3 "" H 1550 1900 50  0001 C CNN
-	1    1550 1900
-	1    0    0    -1
-$EndComp
-Wire Wire Line
-	1650 1950 1650 1800
-Wire Wire Line
-	1650 1800 1550 1800
-Wire Wire Line
-	1700 1850 1700 1700
-Wire Wire Line
-	1700 1700 1550 1700
-Wire Wire Line
-	1750 1750 1750 1600
-Wire Wire Line
-	1750 1600 1550 1600
-Wire Wire Line
-	1800 1650 1800 1500
-Wire Wire Line
-	1800 1500 1550 1500
-Wire Wire Line
-	1650 2050 1650 2200
-Wire Wire Line
-	1650 2200 1550 2200
-Wire Wire Line
-	1700 2150 1700 2300
-Wire Wire Line
-	1700 2300 1550 2300
-Wire Wire Line
-	1750 2250 1750 2400
-Wire Wire Line
-	1750 2400 1550 2400
-Wire Wire Line
-	1800 2350 1800 2500
-Wire Wire Line
-	1800 2500 1550 2500
+F 0 "#PWR015" H 750 2400 50  0001 C CNN
+F 1 "GND" H 755 2477 50  0000 C CNN
+F 2 "" H 750 2650 50  0001 C CNN
+F 3 "" H 750 2650 50  0001 C CNN
+	1    750  2650
+	1    0    0    -1
+$EndComp
 $Comp
 L Device:R_Pack04 RN1
@@
 AR Path="/61DDC3C8/61DB920B" Ref="RN5"  Part="1"
 AR Path="/61DDC5F2/61DB920B" Ref="RN7"  Part="1"
-F 0 "RN1" H 2000 850 50  0000 C CNN
+F 0 "RN5" H 2000 850 50  0000 C CNN
 F 1 "R_Pack04" H 2000 950 50  0000 C CNN
 F 2 "Resistor_SMD:R_Array_Convex_4x0603" V 2325 1250 50  0001 C CNN
@@
 $EndComp
 Wire Wire Line
-	1650 1950 2150 1950
-Wire Wire Line
-	1700 1850 2050 1850
-Wire Wire Line
-	1750 1750 1950 1750
-Wire Wire Line
 	1800 1650 1850 1650
 Wire Wire Line
@@
 Wire Wire Line
 	1950 1450 1950 1750
-Connection ~ 1950 1750
 Wire Wire Line
 	1950 1750 2850 1750
 Wire Wire Line
 	2050 1450 2050 1850
-Connection ~ 2050 1850
 Wire Wire Line
 	2050 1850 2850 1850
@@
 	2150 1950 2850 1950
 Wire Wire Line
-	1800 2350 2550 2350
-Wire Wire Line
-	1750 2250 2450 2250
-Wire Wire Line
-	1700 2150 2350 2150
-Wire Wire Line
-	1650 2050 2250 2050
-Wire Wire Line
 	2250 1450 2250 2050
-Connection ~ 2250 2050
 Wire Wire Line
 	2250 2050 2850 2050
 Wire Wire Line
 	2350 1450 2350 2150
-Connection ~ 2350 2150
 Wire Wire Line
 	2350 2150 2850 2150
 Wire Wire Line
 	2450 1450 2450 2250
-Connection ~ 2450 2250
 Wire Wire Line
 	2450 2250 2850 2250
 Wire Wire Line
 	2550 1450 2550 2350
-Connection ~ 2550 2350
 Wire Wire Line
 	2550 2350 2850 2350
@@
 	2450 1050 2350 1050
 $Comp
-L power:+5V #PWR?
+L power:+5V #PWR06
 U 1 1 61E191BF
 P 1650 1050
-F 0 "#PWR?" H 1650 900 50  0001 C CNN
+AR Path="/61DCCBDC/61E191BF" Ref="#PWR06"  Part="1"
+AR Path="/61DDC172/61E191BF" Ref="#PWR011"  Part="1"
+AR Path="/61DDC3C8/61E191BF" Ref="#PWR016"  Part="1"
+AR Path="/61DDC5F2/61E191BF" Ref="#PWR021"  Part="1"
+F 0 "#PWR016" H 1650 900 50  0001 C CNN
 F 1 "+5V" H 1665 1223 50  0000 C CNN
 F 2 "" H 1650 1050 50  0001 C CNN
@@
 	1    0    0    -1
 $EndComp
+Wire Wire Line
+	1550 2200 1550 2100
+Wire Wire Line
+	1550 2100 750  2100
+Wire Wire Line
+	750  2100 750  2650
+Wire Wire Line
+	1550 1500 1550 1400
+Wire Wire Line
+	1550 1400 750  1400
+Wire Wire Line
+	750  1400 750  2100
+Connection ~ 750  2100
+Wire Wire Line
+	1550 1600 1800 1600
+Wire Wire Line
+	1800 1600 1800 1650
+Wire Wire Line
+	1800 1700 1800 1750
+Wire Wire Line
+	1800 1750 1950 1750
+Connection ~ 1950 1750
+Wire Wire Line
+	1550 1700 1800 1700
+Wire Wire Line
+	1550 1800 1800 1800
+Wire Wire Line
+	1800 1800 1800 1850
+Wire Wire Line
+	1800 1850 2050 1850
+Connection ~ 2050 1850
+Wire Wire Line
+	1550 1900 1800 1900
+Wire Wire Line
+	1800 1900 1800 1950
+Wire Wire Line
+	1800 1950 2150 1950
+Wire Wire Line
+	2250 2050 1800 2050
+Wire Wire Line
+	1800 2050 1800 2300
+Wire Wire Line
+	1800 2300 1550 2300
+Connection ~ 2250 2050
+Wire Wire Line
+	2350 2150 1850 2150
+Wire Wire Line
+	1850 2150 1850 2400
+Wire Wire Line
+	1850 2400 1550 2400
+Connection ~ 2350 2150
+Wire Wire Line
+	2450 2250 1900 2250
+Wire Wire Line
+	1900 2250 1900 2500
+Wire Wire Line
+	1900 2500 1550 2500
+Connection ~ 2450 2250
+Wire Wire Line
+	2550 2350 1950 2350
+Wire Wire Line
+	1950 2350 1950 2600
+Wire Wire Line
+	1950 2600 1550 2600
+Connection ~ 2550 2350
 $EndSCHEMATC
